File: A4/A4.kicad_pcb (KiCad board)
At the start: 2 copper layers, 68.6 x 53.3 mm, 8 parts, among them J1 Power, J2 Digital/PWM, J3 Analog, J4 Digital/PWM

Commit message: PCB 45%
Parts:
- removed J3: Analog, Connector_PinSocket_2.54mm:PinSocket_1x06_P2.54mm_Vertical
- removed J4: Digital/PWM, Connector_PinSocket_2.54mm:PinSocket_1x08_P2.54mm_Vertical
- removed MH1, MH2, MH3, MH4: MountingHole_3.2mm, Arduino_MountingHole:MountingHole_3.2mm
- added A1: Arduino_Nano_v2.x, Module:Arduino_Nano, F.Cu at (121.6, 58.0)
- added BZ1: Buzzer, TerminalBlock_Phoenix:TerminalBlock_Phoenix_MKDS-1,5-2-5.08_1x02_P5.08mm_Horizontal, F.Cu at (154.9, 77.4)
- added J10: LDR/IR, Connector_PinSocket_2.54mm:PinSocket_1x03_P2.54mm_Vertical, F.Cu at (162.8, 63.8)
- added J11: GAS, Connector_PinSocket_2.54mm:PinSocket_1x04_P2.54mm_Vertical, F.Cu at (175.0, 95.8)
- added J12: PIR, Connector_PinSocket_2.54mm:PinSocket_1x03_P2.54mm_Vertical, F.Cu at (167.4, 63.8)
- added J13: Hall Effect, Connector_PinSocket_2.54mm:PinSocket_1x03_P2.54mm_Vertical, F.Cu at (172.0, 63.8)
- added J14: MPU6050, Connector_PinSocket_2.54mm:PinSocket_1x08_P2.54mm_Vertical, F.Cu at (170.4, 73.5)
- added J15: 4x4 Keypad, Connector_PinSocket_2.54mm:PinSocket_1x08_P2.54mm_Vertical, F.Cu at (175.0, 73.5)
- added J16: Joystick, Connector_PinSocket_2.54mm:PinSocket_1x05_P2.54mm_Vertical, F.Cu at (153.6, 97.7)
- added J17: MOTOR, TerminalBlock_Phoenix:TerminalBlock_Phoenix_MKDS-1,5-2-5.08_1x02_P5.08mm_Horizontal, F.Cu at (154.9, 89.5)
- added J5: Servo, Connector_PinSocket_2.54mm:PinSocket_1x03_P2.54mm_Vertical, F.Cu at (153.6, 63.8)
- added J6: Ultrasonic sensor, Connector_PinSocket_2.54mm:PinSocket_1x04_P2.54mm_Vertical, F.Cu at (165.8, 95.8)
- added J7: DHT11, Connector_PinSocket_2.54mm:PinSocket_1x03_P2.54mm_Vertical, F.Cu at (158.2, 63.8)
- added J8: TEST_PIN, Connector_PinSocket_2.54mm:PinSocket_1x02_P2.54mm_Vertical, F.Cu at (158.2, 97.7)
- added J9: 0.96" Oled, Connector_PinSocket_2.54mm:PinSocket_1x04_P2.54mm_Vertical, F.Cu at (170.4, 95.8)
- added POWER_PLUG1: 3V3/5V, Connector_PinSocket_2.54mm:PinSocket_1x03_P2.54mm_Vertical, F.Cu at (176.6, 63.8)
- J1: value Power -> RFID; footprint Connector_PinSocket_2.54mm:PinSocket_1x08_P2.54mm_Vertical -> Connector_PinHeader_2.54mm:PinHeader_1x08_P2.54mm_Vertical
- J2: value Digital/PWM -> I2C 16X2; footprint Connector_PinSocket_2.54mm:PinSocket_1x10_P2.54mm_Vertical -> Connector_PinHeader_2.54mm:PinHeader_1x04_P2.54mm_Vertical
- moved J1 44.9 mm to (165.8, 73.5), turned to 0 degrees
- moved J2 32.8 mm to (86.3, 44.8), turned to 0 degrees
Connections:
- J1 pad 1: unconnected-(J1-Pin_1-Pad1) -> /*10
- J1 pad 2: /IOREF -> /13
- J1 pad 3: /~{RESET} -> /*11
- J1 pad 4: +3V3 -> /12
- J1 pad 5: +5V -> unconnected-(J1-Pin_5-Pad5)
- J1 pad 7: GND -> /*9
- J1 pad 8: VCC -> +3V3
- J2 pad 3: /AREF -> +5V
Other:
- board outline removed
- board text removed: "ICSP"

Commit message: PCB 66%
Parts:
- added J18: Conn_01x01_Pin, Connector_PinHeader_2.54mm:PinHeader_1x01_P2.54mm_Vertical, F.Cu at (118.8, 67.5)
- added J19: Conn_01x01_Pin, Connector_PinHeader_2.54mm:PinHeader_1x01_P2.54mm_Vertical, F.Cu at (222.2, 52.2)
- added J20: Conn_01x01_Pin, Connector_PinHeader_2.54mm:PinHeader_1x01_P2.54mm_Vertical, F.Cu at (194.2, 65.8)
- added J21: Conn_01x01_Pin, Connector_PinHeader_2.54mm:PinHeader_1x01_P2.54mm_Vertical, F.Cu at (236.0, 66.0)
- added J22: Conn_01x01_Pin, Connector_PinHeader_2.54mm:PinHeader_1x01_P2.54mm_Vertical, F.Cu at (264.5, 55.5)
- added J23: Conn_01x01_Pin, Connector_PinHeader_2.54mm:PinHeader_1x01_P2.54mm_Vertical, F.Cu at (115.5, 47.0)
- added J24: Conn_01x01_Pin, Connector_PinHeader_2.54mm:PinHeader_1x01_P2.54mm_Vertical, F.Cu at (180.2, 60.5)
- added J25: Conn_01x01_Pin, Connector_PinHeader_2.54mm:PinHeader_1x01_P2.54mm_Vertical, F.Cu at (125.0, 68.2)
- added J26: Conn_01x01_Pin, Connector_PinHeader_2.54mm:PinHeader_1x01_P2.54mm_Vertical, F.Cu at (122.2, 84.5)
- added J27: Conn_01x01_Pin, Connector_PinHeader_2.54mm:PinHeader_1x01_P2.54mm_Vertical, F.Cu at (248.2, 109.2)
- added J3: TX/RX, Connector_PinHeader_2.54mm:PinHeader_1x04_P2.54mm_Vertical, F.Cu at (185.6, 74.8)
- added J4: Conn_01x01_Pin, Connector_PinHeader_2.54mm:PinHeader_1x01_P2.54mm_Vertical, F.Cu at (99.5, 66.5)
- moved J10 108.8 mm to (263.1, 106.1)
- moved J16 101.9 mm to (240.8, 44.8), turned to 90 degrees
- moved J11 81.4 mm to (253.3, 73.5)
- moved J6 72.4 mm to (226.8, 56.8), turned to 90 degrees
- moved J13 70.4 mm to (239.1, 85.1)
- moved J5 70.0 mm to (218.8, 89.3), turned to 90 degrees
- moved POWER_PLUG1 63.7 mm to (216.1, 113.8), turned to 180 degrees
- moved J12 58.6 mm to (224.6, 76.8), turned to 180 degrees
- moved J9 58.2 mm to (130.1, 53.8), turned to -90 degrees
- moved J1 55.4 mm to (211.3, 41.8)
- moved A1 48.7 mm to (169.1, 69.2)
- moved J14 48.2 mm to (138.2, 37.6), turned to -90 degrees
- moved J2 47.4 mm to (130.3, 62.5), turned to -90 degrees
- moved J7 45.5 mm to (202.8, 72.8), turned to 90 degrees
- moved J15 38.5 mm to (185.6, 36.4)
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Connections:
- J1 pad 1: /*10 -> /13
- J1 pad 2: /13 -> /12
- J1 pad 4: /12 -> /*10
- J10 pad 1: /*9 -> /*11
- J11 pad 2: /*9 -> /*11
- J12 pad 2: /*9 -> /*11
- J13 pad 1: /*9 -> /*11
- J16 pad 1: /*9 -> /*11
- J16 pad 2: /A1 -> /A0
- J16 pad 3: /A0 -> /A1
- J5 pad 1: /*9 -> /*11
- J6 pad 2: /*9 -> /*11
- J7 pad 2: /*9 -> /*11
Routing:
- net VDD: track 0.00 -> 481.1 mm
- net +5V: track 0.00 -> 263.8 mm
- net /*11: track 0.00 -> 254.7 mm
- net /A0: track 0.00 -> 143.5 mm
- net +3V3: track 0.00 -> 138.0 mm
- net /A1: track 0.00 -> 119.1 mm
- net /SCL/A5: track 0.00 -> 99.3 mm
- net GND: track 0.00 -> 77.5 mm
- net /*10: track 0.00 -> 76.4 mm
- net /SDA/A4: track 0.00 -> 72.8 mm
- net /13: track 0.00 -> 62.8 mm
- net /*9: track 0.00 -> 48.8 mm
- net /12: track 0.00 -> 46.8 mm
- net VCC: track 0.00 -> 30.4 mm
- net /RX/0: track 0.00 -> 18.9 mm
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- added copper zone on F.Cu, net GND
Other:
- board outline added: 225.2 x 126.5 mm
- board text added: "PCB TESTER COMMUNITY PROJECT ISA"
